File: mainboard/mainboard.kicad_pcb (KiCad board)
At the start: 2 copper layers, 77 parts, among them J1 Barrel_Jack, J2 USB_C_Receptacle_USB2.0_14P, J3 Conn_01x04, M1 Motor_DC, M2 Motor_DC, M3 Motor_DC, M4 Motor_DC, Q1 2N7002, Q2 2N7002, Q3 2N7002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

Commit message: Added some 3d libs and started routing
Parts:
- added J4: Conn_01x04, Connector_JST:JST_EH_B4B-EH-A_1x04_P2.50mm_Vertical, F.Cu at (87.8, 96.0)
- added R19: 27, Resistor_SMD:R_0603_1608Metric, F.Cu at (82.7, 90.5)
- added R20: 27, Resistor_SMD:R_0603_1608Metric, F.Cu at (82.7, 93.0)
- added REF**: MountingHole_3.2mm_M3, MountingHole:MountingHole_3.2mm_M3, F.Cu at (209.0, 63.0)
- added REF**: MountingHole_3.2mm_M3, MountingHole:MountingHole_3.2mm_M3, F.Cu at (94.0, 63.0)
- added REF**: MountingHole_3.2mm_M3, MountingHole:MountingHole_3.2mm_M3, F.Cu at (118.0, 87.0)
- added REF**: MountingHole_3.2mm_M3, MountingHole:MountingHole_3.2mm_M3, F.Cu at (118.0, 63.0)
- added REF**: MountingHole_3.2mm_M3, MountingHole:MountingHole_3.2mm_M3, F.Cu at (209.0, 87.0)
- added REF**: MountingHole_3.2mm_M3, MountingHole:MountingHole_3.2mm_M3, F.Cu at (94.0, 87.0)
- added TP2: TestPoint_Small, TestPoint:TestPoint_THTPad_1.0x1.0mm_Drill0.5mm, F.Cu at (111.4, 58.2)
- F1: value 10A Poly -> 7A Poly
- L1: footprint LED_THT:LED_D1.8mm_W1.8mm_H2.4mm_Horizontal_O1.27mm_Z1.6mm -> lib:inductor_PA431
- L2: footprint Capacitor_SMD:C_0603_1608Metric -> lib:inductor_BMRx
- R11: value 470 -> 374
- SW2, SW3: footprint lib:SW_SPST_3.3x3.1 -> lib:SW_SPST_2.8x1.9
- TP1, TP3: footprint TestPoint:TestPoint_THTPad_2.0x2.0mm_Drill1.0mm -> TestPoint:TestPoint_THTPad_1.0x1.0mm_Drill0.5mm
- TP4: renamed from TP2; footprint TestPoint:TestPoint_THTPad_2.0x2.0mm_Drill1.0mm -> TestPoint:TestPoint_THTPad_1.0x1.0mm_Drill0.5mm
- moved L2 148.4 mm to (99.4, 55.5)
- moved U5 142.3 mm to (91.8, 54.7), turned to 90 degrees
- moved R6 142.3 mm to (92.6, 52.1)
- moved R5 138.7 mm to (89.4, 52.1)
- moved Q1 138.0 mm to (105.9, 63.1), turned to 90 degrees
- moved C12 137.9 mm to (89.4, 54.8), turned to 90 degrees
- moved R2 137.8 mm to (106.1, 60.6)
- moved U6 131.1 mm to (111.3, 54.1)
- moved R9 128.8 mm to (116.0, 54.4), turned to 180 degrees
- moved TP1 126.3 mm to (108.7, 58.2), turned to 180 degrees
- moved C14 125.7 mm to (113.7, 52.3), turned to 90 degrees
- moved TP3 123.9 mm to (115.3, 56.2), turned to 90 degrees
- moved C13 123.8 mm to (111.1, 51.6)
- moved D2 123.3 mm to (118.0, 56.2)
- moved Q2 122.6 mm to (111.4, 63.1), turned to 90 degrees
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Connections:
- U7 pad 46: USB_D- -> Net-(U7-USB_DM)
- U7 pad 47: USB_D+ -> Net-(U7-USB_DP)
Routing:
- net VBAT: track 0.00 -> 98.3 mm
- net /DISCH_DISABLE: track 0.00 -> 68.5 mm, vias 0 -> 2
- net /vreg_feedback: track 0.00 -> 41.7 mm, vias 0 -> 4
- net PWR_BATT: track 0.00 -> 23.1 mm, vias 0 -> 2
- net VIN: track 0.00 -> 21.7 mm, vias 0 -> 2
- net /CHG_DISABLE: track 0.00 -> 14.9 mm
- net GND: track 0.00 -> 9.38 mm, vias 0 -> 35
- net /CHG_STAT: track 0.00 -> 7.71 mm
- net /CHG_PG: track 0.00 -> 5.94 mm
- net Net-(Q2-G): track 0.00 -> 5.42 mm
- net Net-(U5-EN): track 0.00 -> 3.86 mm
- net Net-(Q1-G): track 0.00 -> 3.51 mm
- net Net-(U6-VSET): track 0.00 -> 3.20 mm
- net Net-(U6-ISET): track 0.00 -> 1.50 mm
- net Net-(D2-A): track 0.00 -> 1.49 mm
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- added copper zone on F.Cu, net +5V
- added copper zone on B.Cu, net GND
- added copper zone on F.Cu, net GND
- added copper zone on F.Cu, net Net-(BT1-+)
- added copper zone on F.Cu, net Net-(U2-SW)
- added copper zone on F.Cu, net Net-(U5-SW)
- added copper zone on F.Cu, net VBAT
- added copper zone on F.Cu, net VIN
Other:
- board outline added: 158.5 x 50 mm
- board text added: "CHG"
- board text added: "PG"
- board text removed: "feedback"
- board text removed: "filtering"

Commit message: More building
Parts:
- added TP7: TestPoint, TestPoint:TestPoint_Pad_D1.0mm, F.Cu at (102.1, 86.5)
- moved R17 23.7 mm to (116.1, 74.9), turned to -90 degrees
- moved R18 21.7 mm to (117.7, 74.9), turned to 90 degrees
- moved C20 18.0 mm to (116.2, 102.8)
- moved D3 17.9 mm to (102.0, 82.7), turned to 90 degrees
- moved C23 16.8 mm to (112.9, 102.7), turned to 180 degrees
- moved SW3 16.2 mm to (109.2, 95.9)
- moved C26 16.2 mm to (113.2, 80.0)
- moved C18 15.0 mm to (109.4, 102.6)
- moved SW2 12.3 mm to (122.1, 77.4), turned to 45 degrees
- moved C25 11.6 mm to (115.8, 82.3), turned to 90 degrees
- moved Y1 11.4 mm to (113.2, 83.0), turned to 90 degrees
- moved C15 11.1 mm to (110.0, 80.5)
- moved U8 11.1 mm to (104.3, 96.1), turned to 180 degrees
- moved R19 9.88 mm to (92.2, 93.3)
- moved R20 9.56 mm to (92.2, 91.7)
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Connections:
- U7 pad 39: unconnected-(U7-GPIO27_ADC1-Pad39) -> Net-(U7-GPIO27_ADC1)
Routing:
- net +3V3: track 0.00 -> 30.9 mm
- net Net-(U7-GPIO26_ADC0): track 0.00 -> 26.5 mm
- net Net-(SW2-A): track 0.00 -> 16.7 mm, vias 0 -> 2
- net +1V1: track 0.00 -> 13.4 mm, vias 0 -> 2
- net Net-(U7-USB_DM): track 0.00 -> 13.3 mm
- net Net-(U7-USB_DP): track 0.00 -> 12.5 mm
- net GND: track 9.38 -> 19.1 mm, vias 35 -> 47
- net /Microcontroller/QSPI_SD3: track 0.00 -> 7.99 mm
- net /Microcontroller/XIN: track 0.00 -> 7.97 mm
- net /Microcontroller/QSPI_SCLK: track 0.00 -> 6.93 mm
- net /Microcontroller/QSPI_CS: track 0.00 -> 6.61 mm
- net /Microcontroller/QSPI_SD0: track 0.00 -> 5.88 mm
- net /Microcontroller/QSPI_SD1: track 0.00 -> 5.26 mm
- net /Microcontroller/QSPI_SD2: track 0.00 -> 4.84 mm
- net VBAT: track 98.3 -> 102.7 mm
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- added copper zone on F.Cu, net +3V3
Other:
- board text removed: "Flash"

Commit message: Finished routing
Parts:
- added J5: Conn_01x04, Connector_PinHeader_1.00mm:PinHeader_1x04_P1.00mm_Vertical, F.Cu at (115.6, 94.2)
- added J6: Conn_01x04, Connector_PinHeader_1.00mm:PinHeader_1x04_P1.00mm_Vertical, F.Cu at (113.3, 89.0)
- added JP1: Jumper_2_Bridged, Jumper:SolderJumper-2_P1.3mm_Bridged_Pad1.0x1.5mm, F.Cu at (206.8, 80.4)
- added JP2: Jumper_2_Bridged, Jumper:SolderJumper-2_P1.3mm_Bridged_Pad1.0x1.5mm, F.Cu at (206.8, 71.9)
- added TP5: TestPoint, TestPoint:TestPoint_Pad_D1.0mm, F.Cu at (106.4, 81.6)
- J2: footprint Connector_USB:USB_C_Receptacle_GCT_USB4105-xx-A_16P_TopMnt_Horizontal -> lib:USB_C_Receptacle_USB2
- moved M1 34.3 mm to (220.0, 89.7), turned to 90 degrees
- moved U4 25.0 mm to (209.8, 70.0), turned to 180 degrees
- moved C20 22.6 mm to (96.0, 92.6), turned to -90 degrees
- moved M2 19.4 mm to (220.0, 80.6), turned to 90 degrees
- moved C11 19.4 mm to (208.8, 81.8), turned to -90 degrees
- moved C23 18.3 mm to (97.6, 92.6), turned to -90 degrees
- moved C5 17.6 mm to (208.8, 73.4), turned to -90 degrees
- moved C10 16.3 mm to (210.7, 81.8), turned to -90 degrees
- moved C4 14.7 mm to (210.7, 73.4), turned to -90 degrees
- moved C19 13.5 mm to (112.3, 92.5), turned to -45 degrees
- moved U3 10.1 mm to (209.8, 78.4), turned to 180 degrees
- moved M4 10.1 mm to (220.0, 62.8), turned to 90 degrees
- moved C18 7.93 mm to (108.1, 94.8), turned to -45 degrees
- moved SW2 5.90 mm to (118.5, 82.0), turned to 0 degrees
- moved M3 4.64 mm to (220.0, 71.7), turned to 90 degrees
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- renumbered TP7 to TP6
Connections:
- D1 pad 1: /CHG_STAT -> CHG_STAT
- D2 pad 1: /CHG_PG -> CHG_PG
- J2 pad A4: unconnected-(J2-VBUS-PadA4)_1 -> VUSB
- J2 pad A9: unconnected-(J2-VBUS-PadA4) -> VUSB
- J2 pad B4: unconnected-(J2-VBUS-PadA4)_2 -> VUSB
- J2 pad B9: unconnected-(J2-VBUS-PadA4)_0 -> VUSB
- SW3 pad 1: GND -> /Microcontroller/QSPI_CS
- SW3 pad 2: /Microcontroller/QSPI_CS -> GND
- TP3 pad 1: /CHG_PG -> CHG_PG
- TP4 pad 1: /CHG_STAT -> CHG_STAT
- U3 pad 11: +3V3 -> Net-(JP1-B)
- U4 pad 11: +3V3 -> Net-(JP2-B)
- U6 pad 5: /CHG_STAT -> CHG_STAT
- U6 pad 6: /CHG_PG -> CHG_PG
- U7 pad 11: unconnected-(U7-GPIO8-Pad11) -> Net-(J5-Pin_1)
- U7 pad 12: unconnected-(U7-GPIO9-Pad12) -> Net-(J5-Pin_2)
- U7 pad 13: unconnected-(U7-GPIO10-Pad13) -> Net-(J5-Pin_3)
- U7 pad 14: unconnected-(U7-GPIO11-Pad14) -> Net-(J5-Pin_4)
- U7 pad 15: unconnected-(U7-GPIO12-Pad15) -> Net-(J6-Pin_1)
- U7 pad 16: unconnected-(U7-GPIO13-Pad16) -> Net-(J6-Pin_2)
- U7 pad 17: unconnected-(U7-GPIO14-Pad17) -> Net-(J6-Pin_3)
- U7 pad 18: unconnected-(U7-GPIO15-Pad18) -> Net-(J6-Pin_4)
- U7 pad 27: /Microcontroller/CHG_STAT -> CHG_STAT
- U7 pad 28: /Microcontroller/CHG_PG -> CHG_PG
- U7 pad 29: unconnected-(U7-GPIO18-Pad29) -> Net-(U7-GPIO18)
Routing:
- net +3V3: track 30.9 -> 178.6 mm, vias 0 -> 7
- net +5V: track 2.07 -> 143.4 mm, vias 0 -> 8
- net MOTC_DIR: track 0.00 -> 127.6 mm
- net MOTC_PWM: track 0.00 -> 127.3 mm
- net MOTD_DIR: track 0.00 -> 127.0 mm
- net MOTD_PWM: track 0.00 -> 126.7 mm
- net MOTA_DIR: track 0.00 -> 122.4 mm
- net MOTA_PWM: track 0.00 -> 122.1 mm
- net MOTB_DIR: track 0.00 -> 121.8 mm
- net MOTB_PWM: track 0.00 -> 121.5 mm
- net CHG_STAT: track 0.00 -> 50.7 mm, vias 0 -> 3
- net CHG_PG: track 0.00 -> 50.0 mm, vias 0 -> 3
- net USB_D-: track 0.00 -> 18.3 mm
- net Net-(M1-+): track 0.00 -> 17.7 mm
- net USB_D+: track 0.00 -> 17.1 mm
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Other:
- board text added: "Back"
- board text added: "Front"
- board text added: "L"
- board text added: "R"
- board text removed: "motors"

Commit message: Trace Edits
Routing:
- net Net-(Q2-G): track 5.42 -> 3.69 mm
Changed lines of the file:
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@@
 		(tags "connector JST EH vertical")
 		(property "Reference" "M4"
-			(at 1.185 -2.11 270)
+			(at 1.185 -2.11 -90)
 			(layer "F.SilkS")
 			(effects
@@
 		)
 		(property "Value" "Motor_DC"
-			(at 1.25 3.400001 270)
+			(at 1.25 3.400001 -90)
 			(layer "F.Fab")
 			(effects
@@
 		)
 		(fp_text user "${REFERENCE}"
-			(at 1.25 1.5 270)
+			(at 1.25 1.5 -90)
 			(layer "F.Fab")
 			(effects
@@
 		(tags "connector JST EH vertical")
 		(property "Reference" "M3"
-			(at 1.235 -2.16 270)
+			(at 1.235 -2.16 -90)
 			(layer "F.SilkS")
 			(effects
@@
 		)
 		(property "Value" "Motor_DC"
-			(at 1.25 3.400001 270)
+			(at 1.25 3.400001 -90)
 			(layer "F.Fab")
 			(effects
@@
 		)
 		(fp_text user "${REFERENCE}"
-			(at 1.25 1.5 270)
+			(at 1.25 1.5 -90)
 			(layer "F.Fab")
 			(effects
@@
 		(tags "connector JST EH vertical")
 		(property "Reference" "M2"
-			(at 1.175 -2.12 270)
+			(at 1.175 -2.12 -90)
 			(layer "F.SilkS")
 			(effects
@@
 		)
 		(property "Value" "Motor_DC"
-			(at 1.25 3.400001 270)
+			(at 1.25 3.400001 -90)
 			(layer "F.Fab")
 			(effects
@@
 		)
 		(fp_text user "${REFERENCE}"
-			(at 1.25 1.5 270)
+			(at 1.25 1.5 -90)
 			(layer "F.Fab")
 			(effects
@@
 		(tags "connector JST EH vertical")
 		(property "Reference" "M1"
-			(at 1.155 -2.17 270)
+			(at 1.155 -2.17 -90)
 			(layer "F.SilkS")
 			(effects
@@
 		)
 		(property "Value" "Motor_DC"
-			(at 1.25 3.400001 270)
+			(at 1.25 3.400001 -90)
 			(layer "F.Fab")
 			(effects
@@
 		)
 		(fp_text user "${REFERENCE}"
-			(at 1.25 1.5 270)
+			(at 1.25 1.5 -90)
 			(layer "F.Fab")
 			(effects
@@
 		(tags "net tie solder jumper bridged")
 		(property "Reference" "JP2"
-			(at 0.000001 -1.46 270)
+			(at 0.000001 -1.46 -90)
 			(layer "F.SilkS")
 			(effects
@@
 		)
 		(property "Value" "Jumper_2_Bridged"
-			(at 0 1.9 270)
+			(at 0 1.9 -90)
 			(layer "F.Fab")
 			(effects
@@
 	)
 	(segment
-		(start 91.05 57.900003)
-		(end 90.95 58.000003)
-		(width 0.2)
-		(layer "B.Cu")
-		(net 6)
-	)
-	(segment
 		(start 91.2 53.15)
 		(end 91 52.95)
@@
 	)
 	(segment
-		(start 88.55 52.1)
-		(end 88.55 52.7)
+		(start 87.1625 54.0875)
+		(end 87.1625 54.4125)
 		(width 0.2)
 		(layer "F.Cu")
@@
 	)
 	(segment
-		(start 87.6 54.65)
-		(end 87.35 54.9)
+		(start 87.1625 54.4125)
+		(end 87.35 54.6)
 		(width 0.2)
 		(layer "F.Cu")
@@
 	)
 	(segment
-		(start 104.275 57.325)
-		(end 106.9 59.95)
+		(start 88.55 52.1)
+		(end 88.55 52.7)
 		(width 0.2)
 		(layer "F.Cu")
@@
 	)
 	(segment
-		(start 87.6 53.65)
-		(end 87.6 54.65)
+		(start 104.275 57.325)
+		(end 106.9 59.95)
 		(width 0.2)
 		(layer "F.Cu")
@@
 	)
 	(segment
-		(start 88.55 52.7)
-		(end 87.6 53.65)
+		(start 87.35 54.6)
+		(end 87.35 54.9)
 		(width 0.2)
 		(layer "F.Cu")
@@
 		(net 7)
 	)
+	(segment
+		(start 88.55 52.7)
+		(end 87.1625 54.0875)
+		(width 0.2)
+		(layer "F.Cu")
+		(net 7)
+	)
 	(via
 		(at 91.05 56.9)
@@
 	(segment
 		(start 110.775 64.15)
-		(end 110.775 64.65)
-		(width 0.2)
-		(layer "F.Cu")
-		(net 34)
-	)
-	(segment
-		(start 110.325 65.1)
-		(end 110.325 65.7)
-		(width 0.2)
-		(layer "F.Cu")
-		(net 34)
-	)
-	(segment
-		(start 110.775 64.65)
-		(end 110.325 65.1)
-		(width 0.2)
-		(layer "F.Cu")
-		(net 34)
-	)
-	(segment
-		(start 110.775 64.15)
 		(end 110.775 62.625)
 		(width 0.2)
@@
 		(polygon
 			(pts
-				(xy 110.5 98.75) (xy 101.95 98.75) (xy 101.95 98.75) (xy 102.525 99.25) (xy 110 99.25)
+				(xy 110.5 98.75) (xy 101.95 98.75) (xy 102.525 99.25) (xy 110 99.25)
 			)
 		)
